Commit message: [add]added meshes

File: urdf/mid360.xacro (robot description, xacro)
@@ -23,6 +23,9 @@
 <xacro:box_inertia m="${length}" w="${width}" d="${length}" h="${height}"/>
   <visual>
+        <!-- <geometry>
+            <box size="${length} ${width} ${height}"/>
+        </geometry> -->
         <geometry>
-            <box size="${length} ${width} ${height}"/>
+            <mesh filename="file://$(find ros2_livox_simulation)/meshes/mid-360.stl" scale="1 1 1"/>
         </geometry>
   </visual>
